File: Canmaster_HW.kicad_sch (KiCad schematic)
At the start: 4 parts, among them M1 Mount_M3, M2 Mount_M3, M3 Mount_M3, M4 Mount_M3

Commit message: Added connection for fault pin. Reversed CAN connector.
Updated some footprints
Other:
- sheet CAN ports: added CAN_SENSE; removed none
- sheet MCU ports: added CAN_SENSE; removed none
Changed lines of the file:
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@@
+    (stroke (width 0) (type default) (color 0 0 0 0))
+  )
+  (wire (pts (xy 95.25 63.5) (xy 105.41 63.5))
     (stroke (width 0) (type default) (color 0 0 0 0))
   )
@@
     (stroke (width 0) (type default) (color 0 0 0 0))
   )
-  (wire (pts (xy 95.25 63.5) (xy 105.41 63.5))
-    (stroke (width 0) (type default) (color 0 0 0 0))
-  )
   (wire (pts (xy 134.62 63.5) (xy 146.05 63.5))
+    (stroke (width 0) (type default) (color 0 0 0 0))
+  )
+  (wire (pts (xy 134.62 74.93) (xy 146.05 74.93))
     (stroke (width 0) (type default) (color 0 0 0 0))
   )
@@
     )
   )
-  (sheet (at 105.41 54.61) (size 29.21 24.13) (fields_autoplaced)
+  (sheet (at 105.41 54.61) (size 29.21 25.4) (fields_autoplaced)
     (stroke (width 0.1524) (type solid) (color 0 0 0 0))
     (fill (color 190 255 175 1.0000))
@@
       (effects (font (size 1.27 1.27)) (justify left bottom))
     )
-    (property "Sheet file" "MCU.kicad_sch" (id 1) (at 105.41 79.3246 0)
+    (property "Sheet file" "MCU.kicad_sch" (id 1) (at 105.41 80.5946 0)
       (effects (font (size 1.27 1.27)) (justify left top))
     )
@@
       (effects (font (size 1.27 1.27)) (justify right))
     )
-    (pin "CAN_TERM_EN" output (at 134.62 72.39 0)
+    (pin "CAN_TERM_EN" output (at 134.62 74.93 0)
       (effects (font (size 1.27 1.27)) (justify right))
     )
@@
       (effects (font (size 1.27 1.27)) (justify right))
     )
-  )
-  (sheet (at 146.05 54.61) (size 26.67 24.13) (fields_autoplaced)
+    (pin "CAN_SENSE" input (at 134.62 72.39 0)
+      (effects (font (size 1.27 1.27)) (justify right))
+    )
+  )
+  (sheet (at 146.05 54.61) (size 26.67 25.4) (fields_autoplaced)
     (stroke (width 0.1524) (type solid) (color 0 0 0 0))
     (fill (color 190 255 175 1.0000))
@@
       (effects (font (size 1.27 1.27)) (justify left bottom))
     )
-    (property "Sheet file" "CAN.kicad_sch" (id 1) (at 146.05 79.3246 0)
+    (property "Sheet file" "CAN.kicad_sch" (id 1) (at 146.05 80.5946 0)
       (effects (font (size 1.27 1.27)) (justify left top))
     )
@@
       (effects (font (size 1.27 1.27)) (justify left))
     )
-    (pin "CAN_TERM_EN" input (at 146.05 72.39 180)
+    (pin "CAN_TERM_EN" input (at 146.05 74.93 180)
+      (effects (font (size 1.27 1.27)) (justify left))
+    )
+    (pin "CAN_SENSE" output (at 146.05 72.39 180)
       (effects (font (size 1.27 1.27)) (justify left))
     )
@@
       (reference "#PWR028") (unit 1) (value "GND") (footprint "")
     )
+    (path "/01b2762a-8576-4e4e-ab62-0edd5e876365/cde0f489-f47b-4ea1-ae42-91b105335d22"
+      (reference "#PWR029") (unit 1) (value "GND") (footprint "")
+    )
     (path "/52e03e0f-0169-4ddc-a0ca-d3b73fdda860/3d4bf2e9-fbaa-44c5-a919-2ca459393bc3"
       (reference "#PWR0101") (unit 1) (value "GND") (footprint "")
@@
       (reference "J2") (unit 1) (value "TC_2030_NL_STLINK") (footprint "N_NonPart:TagConnect_2030_NL")
     )
-    (path "/52e03e0f-0169-4ddc-a0ca-d3b73fdda860/280cbbe2-a1a4-4e26-9cfd-2f52d25a5b4c"
+    (path "/52e03e0f-0169-4ddc-a0ca-d3b73fdda860/ca815669-7de9-4dbd-9580-e40033f02e04"
       (reference "J3") (unit 1) (value "Conn_01x03") (footprint "Connector_Phoenix_MSTB:PhoenixContact_MSTBA_2,5_3-G-5,08_1x03_P5.08mm_Horizontal")
     )
@@
       (reference "R7") (unit 1) (value "120R") (footprint "R_Resistor:R_0603")
     )
+    (path "/01b2762a-8576-4e4e-ab62-0edd5e876365/dc42ea1c-c97f-4a7a-9912-1ce399d8f47b"
+      (reference "R8") (unit 1) (value "10K") (footprint "R_Resistor:R_0603")
+    )
+    (path "/52e03e0f-0169-4ddc-a0ca-d3b73fdda860/e0826cf5-7bc8-46f9-9a4a-faa239d9a3be"
+      (reference "R9") (unit 1) (value "0R") (footprint "R_Resistor:R_0603")
+    )
     (path "/93c82c21-a9a8-4f05-827c-7629e693e47e/999c953d-f873-4181-b275-4a1811787930"
       (reference "U1") (unit 1) (value "USBLC6-4SC6") (footprint "U_IC:SOT23_6")
     )
-    (path "/01b2762a-8576-4e4e-ab62-0edd5e876365/fb416e1c-65b0-4239-b2dc-147ef26ad1d8"
-      (reference "U2") (unit 1) (value "AP2139AK-3.3TRG1") (footprint "U_IC:SOT23_5")
+    (path "/01b2762a-8576-4e4e-ab62-0edd5e876365/47903ef2-65fe-4a97-acb1-9f54a2c16b69"
+      (reference "U2") (unit 1) (value "NCP115ASN330T2G") (footprint "U_IC:SOT23_5")
     )
     (path "/01b2762a-8576-4e4e-ab62-0edd5e876365/8e5e7638-c80b-4d8f-8383-f9fb7b1afade"
