File: MCU.kicad_sch (KiCad schematic)
At the start: 18 parts, among them J2 TC_2030_NL_STLINK, U2 AP2139AK-3.3TRG1, U3 STM32F072CxUx, Y1 ECS-80-12-33-JGN-TR

Commit message: Fix BOOT0 pin being disconnected
Connections:
- net GND: now also U3.44 (BOOT0)
Changed lines of the file:
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@@
+    (stroke (width 0) (type default) (color 0 0 0 0))
+  )
+  (wire (pts (xy 132.08 91.44) (xy 132.08 101.6))
     (stroke (width 0) (type default) (color 0 0 0 0))
   )
@@
     (pin "2")
   )
+  (symbol (lib_id "power:GND") (at 132.08 91.44 180) (unit 1)
+    (in_bom yes) (on_board yes)
+    (property "Reference" "#PWR0102" (id 0) (at 132.08 85.09 0)
+      (effects (font (size 1.27 1.27)) hide)
+    )
+    (property "Value" "GND" (id 1) (at 132.08 87.63 90)
+      (effects (font (size 1.27 1.27)) (justify right))
+    )
+    (property "Footprint" "" (id 2) (at 132.08 91.44 0)
+      (effects (font (size 1.27 1.27)) hide)
+    )
+    (property "Datasheet" "" (id 3) (at 132.08 91.44 0)
+      (effects (font (size 1.27 1.27)) hide)
+    )
+    (pin "1")
+  )
   (symbol (lib_id "DS_LED:DS_0603") (at 220.98 121.92 90) (unit 1)

Commit message: Change RX LED to 220R
Parts:
- R3: value 300R -> 220R
Changed lines of the file:
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@@
       (effects (font (size 1.27 1.27)) (justify left))
     )
-    (property "Value" "300R" (id 1) (at 241.681 113.8998 0)
+    (property "Value" "220R" (id 1) (at 241.681 113.8998 0)
       (effects (font (size 1.27 1.27)) (justify left))
     )

Commit message: Added connection for fault pin. Reversed CAN connector.
Updated some footprints
Parts:
- removed U2: AP2139AK-3.3TRG1, U_IC:SOT23_5, symbol U_Power:AP2139AK-3.3TRG1
- added R8: 10K, R_Resistor:R_0603, symbol R_Resistor:R_0603
- added U2: NCP115ASN330T2G, U_IC:SOT23_5, symbol U_Power:NCP115ASN330T2G
Connections:
- net +3V3: now also U2.5 (VOUT)
- net +5V: now also U2.1 (VIN), U2.3 (EN)
- net GND: now also R8.1, U2.2 (GND)
- net at U3.25 (PB12): now also R8.2
- net CAN_SENSE: now reaches U3.3 (PC14/OSC32_IN)
Other:
- note added: "Version ID pin"
Changed lines of the file:
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@@
+    (stroke (width 0) (type default) (color 0 0 0 0))
+  )
+  (wire (pts (xy 100.33 118.11) (xy 109.22 118.11))
     (stroke (width 0) (type default) (color 0 0 0 0))
   )
@@
     (stroke (width 0) (type default) (color 0 0 0 0))
   )
+  (wire (pts (xy 173.99 140.97) (xy 173.99 142.24))
+    (stroke (width 0) (type default) (color 0 0 0 0))
+  )
   (wire (pts (xy 133.35 48.26) (xy 133.35 50.8))
     (stroke (width 0) (type default) (color 0 0 0 0))
@@
     (stroke (width 0) (type default) (color 0 0 0 0))
   )
+  (wire (pts (xy 171.45 140.97) (xy 173.99 140.97))
+    (stroke (width 0) (type default) (color 0 0 0 0))
+  )
   (wire (pts (xy 217.17 67.31) (xy 233.68 67.31))
     (stroke (width 0) (type default) (color 0 0 0 0))
@@
     (stroke (width 0) (type default) (color 0 0 0 0))
   )
+  (wire (pts (xy 162.56 140.97) (xy 166.37 140.97))
+    (stroke (width 0) (type default) (color 0 0 0 0))
+  )
   (wire (pts (xy 100.33 115.57) (xy 109.22 115.57))
     (stroke (width 0) (type default) (color 0 0 0 0))
+  )
+  (text "Version ID pin" (at 173.99 139.7 0)
+    (effects (font (size 1.27 1.27)) (justify left bottom))
   )
   (label "SWCLK" (at 254 67.31 0)
@@
   (hierarchical_label "CAN_TX" (shape output) (at 138.43 74.93 0)
     (effects (font (size 1.27 1.27)) (justify left))
+  )
+  (hierarchical_label "CAN_SENSE" (shape input) (at 100.33 118.11 180)
+    (effects (font (size 1.27 1.27)) (justify right))
   )
   (hierarchical_label "CAN_MODE" (shape output) (at 100.33 115.57 180)
@@
     (pin "1")
     (pin "2")
+  )
+  (symbol (lib_id "U_Power:NCP115ASN330T2G") (at 67.31 44.45 0) (unit 1)
+    (in_bom yes) (on_board yes) (fields_autoplaced)
+    (property "Reference" "U2" (id 0) (at 67.31 33.5037 0))
+    (property "Value" "NCP115ASN330T2G" (id 1) (at 67.31 36.2788 0))
+    (property "Footprint" "U_IC:SOT23_5" (id 2) (at 76.2 50.8 0)
+      (effects (font (size 1.27 1.27)) hide)
+    )
+    (property "Datasheet" "https://www.diodes.com/assets/Datasheets/AP2138-9.pdf" (id 3) (at 63.47 59.81 0)
+      (effects (font (size 1.27 1.27)) hide)
+    )
+    (property "Params" "3.3V, 300mA" (id 4) (at 67.31 38.3889 0)
+      (effects (font (size 0.6 0.6)))
+    )
+    (pin "1")
+    (pin "2")
+    (pin "3")
+    (pin "4")
+    (pin "5")
   )
   (symbol (lib_id "power:GND") (at 132.08 91.44 180) (unit 1)
@@
     (pin "2")
   )
+  (symbol (lib_id "power:GND") (at 173.99 142.24 0) (unit 1)
+    (in_bom yes) (on_board yes)
+    (property "Reference" "#PWR029" (id 0) (at 173.99 148.59 0)
+      (effects (font (size 1.27 1.27)) hide)
+    )
+    (property "Value" "GND" (id 1) (at 173.99 149.86 90)
+      (effects (font (size 1.27 1.27)) (justify left))
+    )
+    (property "Footprint" "" (id 2) (at 173.99 142.24 0)
+      (effects (font (size 1.27 1.27)) hide)
+    )
+    (property "Datasheet" "" (id 3) (at 173.99 142.24 0)
+      (effects (font (size 1.27 1.27)) hide)
+    )
+    (pin "1")
+  )
+  (symbol (lib_id "R_Resistor:R_0603") (at 168.91 140.97 270) (unit 1)
+    (in_bom yes) (on_board yes) (fields_autoplaced)
+    (property "Reference" "R8" (id 0) (at 168.91 134.1209 90))
+    (property "Value" "10K" (id 1) (at 168.91 136.896 90))
+    (property "Footprint" "R_Resistor:R_0603" (id 2) (at 168.91 138.43 90)
+      (effects (font (size 1.27 1.27)) hide)
+    )
+    (property "Datasheet" "" (id 3) (at 165.1 138.43 0)
+      (effects (font (size 1.27 1.27)) hide)
+    )
+    (property "Size" "R_0603" (id 4) (at 168.91 139.0409 90)
+      (effects (font (size 0.635 0.635)))
+    )
+    (pin "1")
+    (pin "2")
+  )
   (symbol (lib_id "DS_LED:DS_0603") (at 240.03 121.92 90) (unit 1)
     (in_bom yes) (on_board yes) (fields_autoplaced)
@@
     (pin "1")
   )
-  (symbol (lib_id "U_Power:AP2139AK-3.3TRG1") (at 67.31 44.45 0) (unit 1)
-    (in_bom yes) (on_board yes) (fields_autoplaced)
-    (property "Reference" "U2" (id 0) (at 67.31 33.5037 0))
-    (property "Value" "AP2139AK-3.3TRG1" (id 1) (at 67.31 36.2788 0))
-    (property "Footprint" "U_IC:SOT23_5" (id 2) (at 76.2 50.8 0)
-      (effects (font (size 1.27 1.27)) hide)
-    )
-    (property "Datasheet" "https://www.diodes.com/assets/Datasheets/AP2138-9.pdf" (id 3) (at 63.47 59.81 0)
-      (effects (font (size 1.27 1.27)) hide)
-    )
-    (property "Params" "3.3V, 250mA" (id 4) (at 67.31 38.3889 0)
-      (effects (font (size 0.6 0.6)))
-    )
-    (pin "1")
-    (pin "2")
-    (pin "3")
-    (pin "4")
-    (pin "5")
-  )
   (symbol (lib_id "C_Capacitor:C_0603") (at 171.45 45.72 0) (unit 1)

Commit message: Correct LED colors
Parts:
- DS1: value LED,YEL -> LED,RED
Changed lines of the file:
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@@
       (effects (font (size 1.27 1.27)) (justify right))
     )
-    (property "Value" "LED,YEL" (id 1) (at 224.536 123.7423 90)
+    (property "Value" "LED,RED" (id 1) (at 224.536 123.7423 90)
       (effects (font (size 1.27 1.27)) (justify right))
     )
